File: NH3 PCB.kicad_sch (KiCad schematic)
At the start: 9 parts, among them U1 LM393

Commit message: Final Draft for PCB of Ammonia Sensor
Parts:
- added J1: Conn_01x04_Pin, Connector_PinHeader_2.54mm:PinHeader_1x04_P2.54mm_Horizontal, symbol Connector:Conn_01x04_Pin
- C1: footprint (none) -> Capacitor_THT:C_Disc_D5.0mm_W2.5mm_P2.50mm
- D1, D2: footprint (none) -> LED_THT:LED_D5.0mm_Horizontal_O1.27mm_Z3.0mm
- R1, R2: footprint (none) -> Resistor_THT:R_Axial_DIN0207_L6.3mm_D2.5mm_P7.62mm_Horizontal
- RL1: renamed from RL; footprint (none) -> Resistor_THT:R_Axial_DIN0207_L6.3mm_D2.5mm_P7.62mm_Horizontal
- RV1: value ~ -> 500; footprint (none) -> Footprints:NH3Sensor
- RV2: footprint (none) -> Potentiometer_THT:Potentiometer_Bourns_3386X_Horizontal
- U1: footprint (none) -> Footprints:LM393
Connections:
- net Analog Out is gone; now on an unnamed net: C1.2, R1.1, RL1.1, U1.6 (-)
- net +5V: now also RV1.2 (V+), J1.1 (Pin_1)
- net GND: now also J1.4 (Pin_4)
- net at RV1.3 (V-): now also RV1.4 (V-), J1.3 (Pin_3)
- net Digital Out: no longer names the net of R2.1, U1.7
- net Digital Out: now also J1.2 (Pin_2)
